File: rev2/isolated_serial_adapter.kicad_pcb (KiCad board)
At the start: 4 copper layers, 121.2 x 87.1 mm, 104 parts, among them J1 USB_C_Receptacle_USB2.0, J2 RS485_1, J3 RS232, J4 UART_1_FLOW_2, J5 RS485_2, J8 UART_1, J9 UART_1_FLOW_1, SW1 RESET, SW2 FLOW_EN, SW3 VSEL-IN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

Commit message: Final Rev 2 Design
Parts:
- added D9: PWR1, LED_THT:LED_D3.0mm_Clear, F.Cu at (159.5, 60.3)
- added G***: LOGO, slp_logo:sleepylogo_15mm, F.Cu at (158.2, 101.8)
- added R32: 1K, Resistor_SMD:R_0603_1608Metric, F.Cu at (160.8, 66.3)
- added TP1: TestPoint, TestPoint:TestPoint_Pad_D1.0mm, F.Cu at (180.9, 51.5)
- added TP2: TestPoint, TestPoint:TestPoint_Pad_D1.0mm, F.Cu at (170.1, 62.8)
- added TP3: TestPoint, TestPoint:TestPoint_Pad_D1.0mm, F.Cu at (173.9, 47.0)
- added TP4: TestPoint, TestPoint:TestPoint_Pad_D1.0mm, F.Cu at (173.0, 64.7)
- added TP5: TestPoint, TestPoint:TestPoint_Pad_D1.0mm, F.Cu at (167.0, 107.2)
- added TP6: TestPoint, TestPoint:TestPoint_Pad_D1.0mm, F.Cu at (156.1, 107.2)
- added TP7: TestPoint, TestPoint:TestPoint_Pad_D1.0mm, F.Cu at (159.5, 107.2)
- added TP8: TestPoint, TestPoint:TestPoint_Pad_D1.0mm, F.Cu at (170.5, 107.2)
- C18, C22, C3, C4: value 1uF -> 2u2F; footprint Capacitor_SMD:C_0603_1608Metric -> Capacitor_SMD:C_0805_2012Metric
- moved D8 133.2 mm to (111.6, 56.5), turned to -90 degrees
- moved J5 131.2 mm to (106.3, 49.6)
- moved R18 129.6 mm to (123.2, 53.1)
- moved R29 125.1 mm to (114.4, 61.3), turned to 90 degrees
- moved R30 124.6 mm to (108.8, 61.3), turned to 90 degrees
- moved SW6 122.6 mm to (128.2, 46.8), turned to 180 degrees
- moved R13 118.6 mm to (86.3, 56.4), turned to 90 degrees
- moved R19 117.8 mm to (107.8, 56.4), turned to -90 degrees
- moved R28 114.0 mm to (79.6, 61.3), turned to 90 degrees
- moved R27 113.3 mm to (85.2, 61.3), turned to 90 degrees
- moved D6 113.1 mm to (82.4, 56.5), turned to -90 degrees
- moved J2 107.0 mm to (77.2, 49.6)
- moved R16 106.3 mm to (78.6, 56.4), turned to -90 degrees
- moved SW5 101.2 mm to (99.0, 46.8), turned to 180 degrees
- moved C14 96.4 mm to (93.0, 81.3)
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Connections:
- R18 pad 1: Net-(R18-Pad1) -> /RS485/A3
- R18 pad 2: /RS485/B3 -> Net-(R18-Pad2)
- SW6 pad 2: Net-(R18-Pad1) -> Net-(R18-Pad2)
- SW6 pad 3: /RS485/A3 -> /RS485/B3
- U12 pad 2: /UART/RI2_ISO -> /UART/DCD2_ISO
- U12 pad 3: /UART/DCD2_ISO -> /UART/RI2_ISO
- U12 pad 6: /UART/DCD2 -> /UART/RI2
- U12 pad 7: /UART/RI2 -> /UART/DCD2
- U13 pad 1: /UART/DCD2_ISO -> /UART/RI2_ISO
- U13 pad 4: /UART/RI2_ISO -> /UART/DTR2_ISO
- U13 pad 6: /UART/DSR2_ISO -> /UART/RTS2_ISO
- U13 pad 7: /UART/CTS2_ISO -> /UART/DCD2_ISO
- U14 pad 1: /UART/RX2_ISO -> /UART/CTS2_ISO
- U14 pad 4: /UART/DTR2_ISO -> /UART/RX2_ISO
- U14 pad 6: /UART/RTS2_ISO -> /UART/TX2_ISO
- U14 pad 7: /UART/TX2_ISO -> /UART/DSR2_ISO
Routing:
- net +3V3: track 38.7 -> 297.8 mm, vias 13 -> 16
- net +5VD: track 26.4 -> 266.8 mm, vias 11 -> 20
- net /RS485/DIR0: track 3.27 -> 132.6 mm, vias 0 -> 2
- net /RS485/RX0: track 0.00 -> 120.8 mm, vias 0 -> 4
- net /RS485/TX0: track 0.00 -> 114.1 mm, vias 0 -> 4
- net /RS485/RX3: track 0.00 -> 111.8 mm, vias 0 -> 2
- net /RS485/TX3: track 0.00 -> 104.6 mm, vias 0 -> 2
- net /RS485/DIR3: track 4.83 -> 99.3 mm, vias 0 -> 2
- net VDD: track 8.66 -> 69.0 mm, vias 0 -> 14
- net /UART/DSR2: track 0.00 -> 51.1 mm, vias 0 -> 2
- net /UART/RI2: track 0.00 -> 48.8 mm, vias 0 -> 2
- net /UART/DCD2: track 0.00 -> 47.8 mm, vias 0 -> 2
- net /RS232/DSR1: track 14.6 -> 57.0 mm
- net /UART/CTS2: track 0.00 -> 41.6 mm
- net /UART/RTS2: track 0.00 -> 40.0 mm
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- added copper zone on B.Cu, net +3V3
- added copper zone on B.Cu, net +5VD
- added copper zone on B.Cu, net GND
- added copper zone on F.Cu, net GND
- added copper zone on B.Cu, net GND2
- added copper zone on B.Cu, net VDD
- added copper zone on F.Cu, net VDD
- removed copper zone on In2.Cu, net +3V3
- removed copper zone on In2.Cu, net +5VD
Other:
- board size 121.2 x 87.1 mm -> 121.6 x 87.1 mm
- copper layers 4 -> 2
- board text added: "3V3"
- board text added: "5VISO"
- board text added: "ACT"
- board text added: "CH A RS485"
- board text added: "CH B RS232"
- board text added: "CH C UART"
- board text added: "CH D RS485"
- board text added: "DCD RI"
- board text added: "DSR CTS DTR RTS"
- board text added: "FLOW"
- board text added: "GND A B GND"
- board text added: "GND RX TX GND"
- board text added: "JLCJLCJLCJLC"
- board text added: "LVL 2.5 2.7 3.0 3.3 5.0"
- board text added: "ON"
- board text added: "Quad Isolated Serial Adapter"
- board text added: "RS485 TERM"
- board text added: "RST"
- board text added: "RX"
- board text added: "Rev 2"
- board text added: "SW3 R R R R L"
- board text added: "SW4 0 1 2 3 -"
- board text added: "TX"
- board text added: "UART LEVEL"
- board text added: "VBUS"
- board text added: "VDD"
- board text added: "sleepyponylabs.com"
