File: rev2/rs485.kicad_sch (KiCad schematic)
At the start: 22 parts, among them J2 RS485_1, J5 RS485_2, SW5 TERM, SW6 TERM, U5 CA-IS3088WX, U6 CA-IS3088WX

Commit message: Final Rev 2 Design
Connections:
- net A3: now also R18.1; no longer SW6.3 (C)
- net B3: now also SW6.3 (C); no longer R18.2
- net at SW6.2 (B): now also R18.2; no longer R18.1
Other:
- moved on the sheet: R18
Changed lines of the file:
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@@
-    (stroke (width 0) (type default) (color 0 0 0 0))
-  )
-  (wire (pts (xy 156.21 124.46) (xy 171.45 124.46))
     (stroke (width 0) (type default) (color 0 0 0 0))
   )
@@
     (stroke (width 0) (type default) (color 0 0 0 0))
   )
+  (wire (pts (xy 171.45 130.81) (xy 171.45 132.08))
+    (stroke (width 0) (type default) (color 0 0 0 0))
+  )
   (wire (pts (xy 80.01 139.7) (xy 91.44 139.7))
     (stroke (width 0) (type default) (color 0 0 0 0))
@@
     (stroke (width 0) (type default) (color 0 0 0 0))
   )
-  (wire (pts (xy 156.21 124.46) (xy 156.21 134.62))
-    (stroke (width 0) (type default) (color 0 0 0 0))
-  )
   (wire (pts (xy 208.28 135.89) (xy 208.28 138.43))
     (stroke (width 0) (type default) (color 0 0 0 0))
@@
     (stroke (width 0) (type default) (color 0 0 0 0))
   )
-  (wire (pts (xy 171.45 140.97) (xy 171.45 142.24))
+  (wire (pts (xy 144.78 142.24) (xy 171.45 142.24))
     (stroke (width 0) (type default) (color 0 0 0 0))
   )
@@
     (stroke (width 0) (type default) (color 0 0 0 0))
   )
+  (wire (pts (xy 171.45 140.97) (xy 156.21 140.97))
+    (stroke (width 0) (type default) (color 0 0 0 0))
+  )
   (wire (pts (xy 190.5 66.04) (xy 203.2 66.04))
     (stroke (width 0) (type default) (color 0 0 0 0))
@@
     (stroke (width 0) (type default) (color 0 0 0 0))
   )
+  (wire (pts (xy 156.21 140.97) (xy 156.21 134.62))
+    (stroke (width 0) (type default) (color 0 0 0 0))
+  )
   (wire (pts (xy 156.21 58.42) (xy 156.21 63.5))
     (stroke (width 0) (type default) (color 0 0 0 0))
@@
     (stroke (width 0) (type default) (color 0 0 0 0))
   )
+  (wire (pts (xy 171.45 121.92) (xy 171.45 123.19))
+    (stroke (width 0) (type default) (color 0 0 0 0))
+  )
   (wire (pts (xy 88.9 129.54) (xy 88.9 142.24))
     (stroke (width 0) (type default) (color 0 0 0 0))
   )
+  (wire (pts (xy 171.45 142.24) (xy 171.45 140.97))
+    (stroke (width 0) (type default) (color 0 0 0 0))
+  )
   (polyline (pts (xy 231.14 162.56) (xy 106.68 162.56))
     (stroke (width 0) (type default) (color 0 0 0 0))
@@
     (stroke (width 0) (type default) (color 0 0 0 0))
   )
-  (wire (pts (xy 144.78 142.24) (xy 171.45 142.24))
-    (stroke (width 0) (type default) (color 0 0 0 0))
-  )
   (wire (pts (xy 203.2 142.24) (xy 203.2 133.35))
     (stroke (width 0) (type default) (color 0 0 0 0))
   )
-  (wire (pts (xy 171.45 132.08) (xy 171.45 133.35))
-    (stroke (width 0) (type default) (color 0 0 0 0))
-  )
   (wire (pts (xy 144.78 66.04) (xy 171.45 66.04))
-    (stroke (width 0) (type default) (color 0 0 0 0))
-  )
-  (wire (pts (xy 171.45 124.46) (xy 171.45 121.92))
     (stroke (width 0) (type default) (color 0 0 0 0))
   )
@@
     (pin "1")
   )
-  (symbol (lib_id "Device:R") (at 171.45 137.16 0) (unit 1)
-    (in_bom yes) (on_board yes) (fields_autoplaced)
-    (property "Reference" "R18" (id 0) (at 173.99 135.8899 0)
-      (effects (font (size 1.27 1.27)) (justify left))
-    )
-    (property "Value" "120R" (id 1) (at 173.99 138.4299 0)
-      (effects (font (size 1.27 1.27)) (justify left))
-    )
-    (property "Footprint" "Resistor_SMD:R_0603_1608Metric" (id 2) (at 169.672 137.16 90)
-      (effects (font (size 1.27 1.27)) hide)
-    )
-    (property "Datasheet" "~" (id 3) (at 171.45 137.16 0)
+  (symbol (lib_id "Device:R") (at 171.45 127 0) (unit 1)
+    (in_bom yes) (on_board yes) (fields_autoplaced)
+    (property "Reference" "R18" (id 0) (at 173.99 125.7299 0)
+      (effects (font (size 1.27 1.27)) (justify left))
+    )
+    (property "Value" "120R" (id 1) (at 173.99 128.2699 0)
+      (effects (font (size 1.27 1.27)) (justify left))
+    )
+    (property "Footprint" "Resistor_SMD:R_0603_1608Metric" (id 2) (at 169.672 127 90)
+      (effects (font (size 1.27 1.27)) hide)
+    )
+    (property "Datasheet" "~" (id 3) (at 171.45 127 0)
       (effects (font (size 1.27 1.27)) hide)
     )
@@
   (symbol (lib_id "Switch:SW_SPDT") (at 162.56 132.08 0) (mirror y) (unit 1)
     (in_bom yes) (on_board yes)
-    (property "Reference" "SW6" (id 0) (at 162.56 137.16 0))
-    (property "Value" "TERM" (id 1) (at 162.56 139.7 0))
+    (property "Reference" "SW6" (id 0) (at 162.56 124.46 0))
+    (property "Value" "TERM" (id 1) (at 162.56 127 0))
     (property "Footprint" "Button_Switch_THT:SW_CuK_OS102011MA1QN1_SPDT_Angled" (id 2) (at 162.56 132.08 0)
       (effects (font (size 1.27 1.27)) hide)
