File: rev2/uart.kicad_sch (KiCad schematic)
At the start: 11 parts, among them J4 UART_1_FLOW_2, J8 UART_1, J9 UART_1_FLOW_1, U10 CA-IS3763HW, U12 CA-IS3720HG, U13 SRDA05-4BTG, U14 SRDA05-4BTG

Commit message: Final Rev 2 Design
Connections:
- net CTS2_ISO: now also U14.1 (IN1); no longer U13.7 (IN4)
- net DCD2: now also U12.7 (VOA); no longer U12.6 (VOB)
- net DCD2_ISO: now also U12.2 (VIA), U13.7 (IN4); no longer U12.3 (VIB), U13.1 (IN1)
- net DSR2_ISO: now also U14.7 (IN4); no longer U13.6 (IN3)
- net DTR2_ISO: now also U13.4 (IN2); no longer U14.4 (IN2)
- net RI2: now also U12.6 (VOB); no longer U12.7 (VOA)
- net RI2_ISO: now also U12.3 (VIB), U13.1 (IN1); no longer U12.2 (VIA), U13.4 (IN2)
- net RTS2_ISO: now also U13.6 (IN3); no longer U14.6 (IN3)
- net RX2_ISO: now also U14.4 (IN2); no longer U14.1 (IN1)
- net TX2_ISO: now also U14.6 (IN3); no longer U14.7 (IN4)
